File: pcb/mSD-Shield_v20.brd (EAGLE design)
At the start: 65.4 x 53.3 mm, 63 parts, among them IC1 74LVC244, IC2 DS1307, Q1 32kHz, Q1B 32kHz, U1 TS5204, X1 PASSER, X2 PASSER, X3 PASSER, X4 PASSER, X5 MICRO-SD

Commit message: updated schematic and layout files
Parts:
- U1: value TS5204 -> TS5204-3V3
Changed lines of the file:
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@@
 <?xml version="1.0" encoding="utf-8"?>
 <!DOCTYPE eagle SYSTEM "eagle.dtd">
-<eagle version="6.5.0">
+<eagle version="6.6.0">
 <drawing>
 <settings>
@@
 </autorouter>
 <elements>
-<element name="U1" library="Voltage-Reg" package="SOT23" value="TS5204" x="27.94" y="21.59" smashed="yes" rot="R270">
+<element name="U1" library="Voltage-Reg" package="SOT23" value="TS5204-3V3" x="27.94" y="21.59" smashed="yes" rot="R270">
 <attribute name="NAME" x="29.845" y="22.5425" size="0.8128" layer="25" font="vector" ratio="10" rot="R270"/>
 <attribute name="VALUE" x="30.7975" y="23.8125" size="0.8128" layer="27" font="vector" ratio="10" rot="R270"/>
