File: pcb/mSD-Shield_v20.sch (EAGLE design)
At the start: 63 parts, among them IC1 74LVC244, IC2 DS1307, Q1 32kHz, Q1B 32kHz, U1 TS5204, X1 PASSER, X2 PASSER, X3 PASSER, X4 PASSER, X5 MICRO-SD

Commit message: updated schematic and layout files
Parts:
- U1: value TS5204 -> TS5204-3V3
Changed lines of the file:
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@@
 <?xml version="1.0" encoding="utf-8"?>
 <!DOCTYPE eagle SYSTEM "eagle.dtd">
-<eagle version="6.5.0">
+<eagle version="6.6.0">
 <drawing>
 <settings>
@@
 </classes>
 <parts>
-<part name="U1" library="Voltage-Reg" deviceset="TS5204" device=""/>
+<part name="U1" library="Voltage-Reg" deviceset="TS5204" device="" value="TS5204-3V3"/>
 <part name="GND9" library="supply1" deviceset="GND" device=""/>
 <part name="C1" library="rcl" deviceset="C-EU" device="C0805" value="2uF"/>
