File: pcb/mSD-Shield_v20.sch (EAGLE design)
At the start: 63 parts, among them IC1 74LVC244, IC2 DS1307, Q1 32kHz, Q1B 32kHz, U1 TS5204-3V3, X1 PASSER, X2 PASSER, X3 PASSER, X4 PASSER, X5 MICRO-SD

Commit message: cleaned up schematics and layout
Changed lines of the file:
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@@
 <setting verticaltext="up"/>
 </settings>
-<grid distance="0.1" unitdist="inch" unit="inch" style="lines" multiple="1" display="no" altdistance="0.01" altunitdist="inch" altunit="inch"/>
+<grid distance="0.05" unitdist="inch" unit="inch" style="lines" multiple="1" display="yes" altdistance="0.025" altunitdist="inch" altunit="inch"/>
 <layers>
 <layer number="1" name="Top" color="4" fill="1" visible="no" active="no"/>
@@
 <part name="GND5" library="supply1" deviceset="GND" device=""/>
 <part name="C5" library="rcl" deviceset="C-EU" device="C0603" value="2uF"/>
-<part name="FRAME1" library="frames" deviceset="A4L-LOC" device=""/>
 <part name="IC1" library="74xx-eu" deviceset="74*244" device="DW" technology="HC" value="74LVC244"/>
 <part name="GND10" library="supply1" deviceset="GND" device=""/>
@@
 <part name="LCD_SCL" library="jumper" deviceset="SJ" device=""/>
 <part name="LCD_SDA" library="jumper" deviceset="SJ" device=""/>
+<part name="FRAME1" library="we-symbol" deviceset="FRAME-A4L" device=""/>
 </parts>
 <sheets>
@@
 <wire x1="88.265" y1="17.78" x2="90.297" y2="17.78" width="0.8128" layer="94"/>
 <wire x1="77.47" y1="80.01" x2="75.438" y2="80.01" width="0.8128" layer="94"/>
-<text x="162.56" y="31.75" size="1.27" layer="95">Released under the Creative Commons Attribution Share-Alike License</text>
-<text x="162.56" y="29.21" size="1.27" layer="95">http://creativecommons.org/licenses/by-sa/4.0/</text>
-<text x="162.56" y="25.4" size="1.27" layer="95">Designed by Andreas Watterott (Watterott electronic)</text>
+<text x="162.56" y="21.59" size="1.27" layer="95">Released under the Creative Commons Attribution Share-Alike License</text>
+<text x="162.56" y="19.05" size="1.27" layer="95">http://creativecommons.org/licenses/by-sa/4.0/</text>
+<text x="162.56" y="15.24" size="1.27" layer="95">Designed by Andreas Watterott (Watterott electronic)</text>
 <text x="46.99" y="105.41" size="1.778" layer="95">(EthShield uses 2, 4, 10_SS)</text>
 <text x="30.48" y="76.2" size="1.27" layer="95" rot="R180">LCD_LED/GPIO</text>
@@
 <attribute name="VALUE" x="148.082" y="10.541" size="1.778" layer="96"/>
 </instance>
-<instance part="FRAME1" gate="G$1" x="0" y="0" smashed="yes">
-<attribute name="DRAWING_NAME" x="217.17" y="15.24" size="2.54" layer="94" font="vector"/>
-<attribute name="LAST_DATE_TIME" x="217.17" y="10.16" size="2.286" layer="94" font="vector"/>
-<attribute name="SHEET" x="230.505" y="5.08" size="2.54" layer="94" font="vector"/>
-</instance>
 <instance part="IC1" gate="A" x="172.72" y="85.09" smashed="yes" rot="MR0">
 <attribute name="NAME" x="180.34" y="93.345" size="1.778" layer="95" rot="MR0"/>
@@
 <attribute name="VALUE" x="19.05" y="132.08" size="1.778" layer="96" rot="MR90"/>
 </instance>
-<instance part="X1" gate="G$1" x="166.37" y="19.05"/>
-<instance part="X2" gate="G$1" x="173.99" y="19.05"/>
-<instance part="X3" gate="G$1" x="181.61" y="19.05"/>
-<instance part="X4" gate="G$1" x="189.23" y="19.05"/>
+<instance part="X1" gate="G$1" x="165.1" y="7.62" smashed="yes"/>
+<instance part="X2" gate="G$1" x="170.18" y="7.62" smashed="yes"/>
+<instance part="X3" gate="G$1" x="175.26" y="7.62" smashed="yes"/>
+<instance part="X4" gate="G$1" x="180.34" y="7.62" smashed="yes"/>
 <instance part="0" gate="P" x="90.17" y="161.29" smashed="yes" rot="R180">
 <attribute name="NAME" x="92.202" y="160.6042" size="1.778" layer="95"/>
@@
 </instance>
 <instance part="BAT" gate="G$1" x="215.9" y="46.99"/>
-<instance part="LOGO2" gate="G$1" x="201.93" y="19.05"/>
-<instance part="LOGO3" gate="G$1" x="201.93" y="11.43"/>
+<instance part="LOGO2" gate="G$1" x="208.28" y="7.62"/>
+<instance part="LOGO3" gate="G$1" x="198.12" y="7.62"/>
 <instance part="RESET" gate="G$1" x="30.48" y="135.89" smashed="yes" rot="MR270">
 <attribute name="NAME" x="26.67" y="132.715" size="1.778" layer="95" rot="MR180"/>
@@
 <attribute name="VALUE" x="52.07" y="49.53" size="1.778" layer="96" rot="MR180"/>
 </instance>
+<instance part="FRAME1" gate="G$1" x="0" y="0"/>
 </instances>
 <busses>
